File: active-filter/active-fiter.kicad_pcb (KiCad board)
At the start: 2 copper layers, 43 parts, among them J1 AudioJack2_Switch, J10 Conn_01x03, J2 AudioJack2_Switch, J3 AudioJack2_Switch, J4 AudioJack2_Switch, J5 AudioJack2_Switch, J6 AudioJack2_Switch, J7 AudioJack2_Switch, J8 AudioJack2_Switch, J9 AudioJack2_Switch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

Commit message: Add active filter pcb
Parts:
- removed J1, J2, J3, J4, J5, J6, J7, J8, J9: AudioJack2_Switch, Connector_Audio:Jack_6.35mm_Neutrik_NMJ4HHD2_Horizontal
- added J11: Conn_01x03, Connector_JST:JST_PH_B3B-PH-K_1x03_P2.00mm_Vertical, F.Cu at (239.9, 117.6)
- added J12: AudioJack3_SwitchTR, Connector_Audio:Jack_3.5mm_CUI_SJ1-3525N_Horizontal, F.Cu at (158.6, 120.9)
- added J13: AudioJack3_SwitchTR, Connector_Audio:Jack_3.5mm_CUI_SJ1-3525N_Horizontal, F.Cu at (173.9, 120.9)
- added J14: AudioJack3_SwitchTR, Connector_Audio:Jack_3.5mm_CUI_SJ1-3525N_Horizontal, F.Cu at (189.3, 120.9)
- added J15: AudioJack3_SwitchTR, Connector_Audio:Jack_3.5mm_CUI_SJ1-3525N_Horizontal, F.Cu at (205.0, 121.1)
- added J16: AudioJack3_SwitchTR, Connector_Audio:Jack_3.5mm_CUI_SJ1-3525N_Horizontal, F.Cu at (205.0, 30.0)
- added J17: AudioJack3_SwitchTR, Connector_Audio:Jack_3.5mm_CUI_SJ1-3525N_Horizontal, F.Cu at (189.5, 30.0)
- added J18: AudioJack3_SwitchTR, Connector_Audio:Jack_3.5mm_CUI_SJ1-3525N_Horizontal, F.Cu at (174.0, 30.0)
- added J19: AudioJack3_SwitchTR, Connector_Audio:Jack_3.5mm_CUI_SJ1-3525N_Horizontal, F.Cu at (158.5, 30.0)
- added J20: AudioJack3_SwitchTR, Connector_Audio:Jack_3.5mm_CUI_SJ1-3525N_Horizontal, F.Cu at (246.4, 74.9)
- C1, C2: footprint Capacitor_THT:CP_Axial_L18.0mm_D10.0mm_P25.00mm_Horizontal -> Capacitor_THT:CP_Radial_D10.0mm_P5.00mm
- moved C1 204.4 mm to (239.9, 101.0)
- moved R4 197.9 mm to (237.7, 54.9), turned to 90 degrees
- moved C2 193.9 mm to (227.8, 101.0)
- moved R6 190.4 mm to (231.6, 54.9), turned to 90 degrees
- moved R5 184.9 mm to (225.6, 53.8), turned to -90 degrees
- moved R3 180.6 mm to (219.2, 53.8), turned to -90 degrees
- moved R21 175.4 mm to (219.3, 91.2), turned to 90 degrees
- moved C3 173.1 mm to (230.6, 84.6), turned to 180 degrees
- moved R12 165.6 mm to (208.7, 65.5), turned to -90 degrees
- moved U1 165.4 mm to (224.5, 71.4)
- moved R20 164.8 mm to (208.8, 85.1), turned to 90 degrees
- moved J10 162.9 mm to (228.8, 117.6)
- moved R10 160.0 mm to (201.8, 66.0), turned to 90 degrees
- moved R16 159.1 mm to (201.8, 84.6), turned to -90 degrees
- moved R11 151.1 mm to (193.5, 65.5), turned to -90 degrees
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Routing:
- net Net-(U1--): track 0.00 -> 144.1 mm
- net Net-(U1-+): track 0.00 -> 128.6 mm
- net VDD: track 0.00 -> 90.7 mm
- net Net-(J20-PadR): track 0.00 -> 62.6 mm
- net VEE: track 0.00 -> 56.1 mm
- net Net-(R3-Pad2): track 0.00 -> 43.9 mm
- net Net-(R13-Pad2): track 0.00 -> 20.0 mm
- net Net-(R11-Pad1): track 0.00 -> 20.0 mm
- net Net-(R15-Pad2): track 0.00 -> 20.0 mm
- net Net-(R1-Pad2): track 0.00 -> 20.0 mm
- net Net-(R16-Pad2): track 0.00 -> 19.9 mm
- net Net-(R7-Pad2): track 0.00 -> 19.8 mm
- net Net-(R14-Pad2): track 0.00 -> 19.8 mm
- net Net-(R10-Pad2): track 0.00 -> 19.7 mm
- net Net-(R14-Pad1): track 0.00 -> 18.6 mm
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- added copper zone on B.Cu, net GND
Other:
- board outline added: 100.1 x 100.1 mm
