File: active-filter/active-fiter.kicad_sch (KiCad schematic)
At the start: 43 parts, among them J1 AudioJack2_Switch, J10 Conn_01x03, J2 AudioJack2_Switch, J3 AudioJack2_Switch, J4 AudioJack2_Switch, J5 AudioJack2_Switch, J6 AudioJack2_Switch, J7 AudioJack2_Switch, J8 AudioJack2_Switch, J9 AudioJack2_Switch, U1 LM318N

Commit message: Add active filter pcb
Parts:
- removed J1, J2, J3, J4, J5, J6, J7, J8, J9: AudioJack2_Switch, Connector_Audio:Jack_6.35mm_Neutrik_NMJ4HHD2_Horizontal, symbol Connector_Audio:AudioJack2_Switch
- added J11: Conn_01x03, Connector_JST:JST_PH_B3B-PH-K_1x03_P2.00mm_Vertical, symbol Connector_Generic:Conn_01x03
- added J12, J13, J14, J15, J16, J17, J18, J19, J20: AudioJack3_SwitchTR, Connector_Audio:Jack_3.5mm_CUI_SJ1-3525N_Horizontal, symbol Connector_Audio:AudioJack3_SwitchTR
- C1, C2: footprint Capacitor_THT:CP_Axial_L18.0mm_D10.0mm_P25.00mm_Horizontal -> Capacitor_THT:CP_Radial_D10.0mm_P5.00mm
Connections:
- net GND: now also J11.2 (Pin_2), J12.RN, J12.S, J12.TN, J13.RN, J13.S, J13.TN, J14.RN, J14.S, J14.TN, J15.RN, J15.S, J15.TN, J16.RN, J16.S, J16.TN, J17.RN, J17.S, J17.TN, J18.RN, J18.S, J18.TN, J19.RN, J19.S, J19.TN, J20.RN, J20.S, J20.TN
- net VDD: now also J11.1 (Pin_1)
- net VEE: now also J11.3 (Pin_3)
- net at RV14.1: now also J13.R, J13.T
- net at RV15.1: now also J14.R, J14.T
- net at R4.2, R6.2, U1.6: now also J20.R, J20.T
- net at RV13.1: now also J12.R, J12.T
- net at RV9.1: now also J19.R, J19.T
- net at RV10.1: now also J18.R, J18.T
- net at RV11.1: now also J17.R, J17.T
- net at RV16.1: now also J15.R, J15.T
- net at RV12.1: now also J16.R, J16.T
