File: amplifier/amplifier.kicad_sch (KiCad schematic)
At the start: 14 parts, among them J1 AudioJack3_SwitchTR, J2 Conn_01x02, Q1 NMOS

Commit message: Add amplifier pcb
Parts:
- removed Q1: NMOS, symbol Simulation_SPICE:NMOS
- added C7: C_Polarized, Capacitor_THT:CP_Radial_D16.0mm_P7.50mm, symbol Device:C_Polarized
- added J3: Conn_01x02, Connector_AMASS:AMASS_XT30PW-M_1x02_P2.50mm_Horizontal, symbol Connector_Generic:Conn_01x02
- added Q2: Q_NMOS_GDS, Package_TO_SOT_THT:TO-247-3_Vertical, symbol Transistor_FET:Q_NMOS_GDS
- added Q3: Q_NMOS_GDS, Package_TO_SOT_THT:TO-220-3_Vertical, symbol Transistor_FET:Q_NMOS_GDS
- added R4: R, Resistor_THT:R_Axial_Power_L75.0mm_W9.0mm_P86.36mm, symbol Device:R
- C1, C6: footprint (none) -> Capacitor_THT:C_Disc_D4.7mm_W2.5mm_P5.00mm
- C2: footprint (none) -> Capacitor_THT:C_Radial_D10.0mm_H20.0mm_P5.00mm
- C3: footprint (none) -> Capacitor_THT:C_Rect_L33.0mm_W13.0mm_P27.50mm_MKS4
- C4, C5: footprint (none) -> Capacitor_THT:CP_Radial_D16.0mm_P7.50mm
- J1: footprint (none) -> Connector_Audio:Jack_3.5mm_CUI_SJ1-3525N_Horizontal
- J2: footprint (none) -> Connector_JST:JST_NV_B02P-NV_1x02_P5.00mm_Vertical
- R1, R2: footprint (none) -> Resistor_THT:R_Axial_DIN0207_L6.3mm_D2.5mm_P15.24mm_Horizontal
- R3: footprint (none) -> Resistor_THT:R_Axial_Power_L75.0mm_W9.0mm_P86.36mm
- RV1, RV2: footprint (none) -> Potentiometer_THT:Potentiometer_Bourns_PTV09A-1_Single_Vertical
Connections:
- net GND: now also C5.2, C6.2, C7.2, J3.2 (Pin_2), Q2.3 (S), Q3.3 (S)
- net VDD: now also C7.1, J3.1 (Pin_1), R4.1
- net at C3.1, C4.1, R3.2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: now also Q2.2 (D), Q3.2 (D), R4.2
- net at R1.2, R2.2: now also Q2.1 (G), Q3.1 (G)
